Commit message: Add Stretch 4 PG4 gripper model + Fix limit in SG4

File: roboplan_example_models/models/stretch4_robot_model/stretch4_sg4.urdf (robot description, URDF)
Before this commit: robot stretch, 53 links, 52 joints
Joints:
- joint wrist_pitch_joint: limit lower=-4.276 upper=1.135 effort=0 velocity=1.0 -> lower=-1.135 upper=4.276 effort=0 velocity=1.0
